File: board/bleriot-relay.kicad_pcb (KiCad board)
At the start: 2 copper layers, 80 x 40 mm, 29 parts, among them J1 TX, U1 PAN2110P0AA, U2 PY32F003W1xSx, U3 PSU, U4 LM1117MP-3.3, U5 MOC306XMS, X1 SWD, Y1 16MHz

Commit message: WIP
Other:
- board text added: "230V~ 2A max."
- board text added: "GND SENS +5V"
- board text added: "L ~{IN} N"
- board text added: "L ~{OUT} N"
Changed lines of the file:
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@@
 		(tags "capacitor")
 		(property "Reference" "C7"
-			(at 0 -1.68 90)
+			(at 3 0 90)
 			(layer "F.SilkS")
 			(effects
@@
 		(tags "capacitor")
 		(property "Reference" "C6"
-			(at 0 1.5 90)
+			(at 3 0 90)
 			(layer "F.SilkS")
 			(effects
@@
 		(tags "capacitor")
 		(property "Reference" "C5"
-			(at 0 -1.5 90)
+			(at 3 0 90)
 			(layer "F.SilkS")
 			(effects
@@
 		(layer "Edge.Cuts")
 	)
+	(gr_text "GND  SENS  +5V"
+		(at 163 71.5 90)
+		(layer "F.SilkS")
+		(effects
+			(font
+				(size 1 1)
+				(thickness 0.15)
+			)
+			(justify top)
+		)
+	)
+	(gr_text "L ~{OUT} N"
+		(at 87 59.5 270)
+		(layer "F.SilkS")
+		(effects
+			(font
+				(size 1 1)
+				(thickness 0.15)
+			)
+			(justify top)
+		)
+	)
+	(gr_text "L ~{IN} N"
+		(at 87 73.5 270)
+		(layer "F.SilkS")
+		(effects
+			(font
+				(size 1 1)
+				(thickness 0.15)
+			)
+			(justify top)
+		)
+	)
+	(gr_text "230V~\n2A max."
+		(at 87.5 49 270)
+		(layer "F.SilkS")
+		(effects
+			(font
+				(size 1.2 1.2)
+				(thickness 0.2)
+			)
+		)
+	)
 	(gr_text "BLERIOT RELAY v1.0"
-		(at 88 47 0)
+		(at 101.5 47 0)
 		(layer "F.SilkS")
 		(effects
